File: PCB/PCB KiCad/power.kicad_sch (KiCad schematic)
At the start: 11 parts, among them U3 LM285D-2.5, U4 AMS1117-3.3

Commit message: Updated IR emitter resistor values & alternative supply sources
The resistor values for the IR emitters in DB2.1 schematics were too high. Some of the emitters didn't even lit up.

I added new resistor values for the maximum forward current the emitters can handle. One option would be to balance the resistances for equal electrical output power of the emitters, but I haven't done research on what the actual optical output power would in that case be. In other words, if one would like the emitters lit the plastic sample with equal power. Please note, that the package of D4 and D5 is NOT 1206 and that they have a higher forward current than the other emitters.

The version number on the schematics is changed to 2.1.1. Please correct this, if it is wrong.

There are also alternative supply sources for the hard-to-get TI components and the 3.3V voltage regulator. These "clones" are tested and they seem to work, but I can't compare the signal quality to the original components since the stocks at official distributors are empty.
Parts:
- U4: Supplier (none) -> https://www.aliexpress.com/item/33049686463.html
Changed lines of the file:
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@@
   (title_block
     (title "Development Board")
-    (date "2022-03-15")
-    (rev "2.1")
+    (date "2023-01-23")
+    (rev "2.1.1")
     (company "Plastic Scanner")
   )
@@
       (effects (font (size 1.27 1.27)) hide)
     )
+    (property "Supplier" "https://www.aliexpress.com/item/33049686463.html" (id 4) (at 189.23 63.5 0)
+      (effects (font (size 1.27 1.27)) hide)
+    )
